File: boards/double_in_cab_breakout/double_in_cab_breakout.sch (KiCad schematic (older format))
At the start: 10 parts, among them P10 CONN_JST_PH_2, P100 CONN_TERM_BLOCK_2POS_3P5MM, P101 CONN_TERM_BLOCK_2POS_3P5MM, P11 CONN_JST_PH_2, P13 CONN_JST_PH_2, P14 CONN_JST_PH_2, P16 CONN_JST_PH_2, P17 CONN_JST_PH_2

Commit message: Modifications
Parts:
- added R1001: RES_0_0P_1V4_1206, symbol RES_0_0P_1V4_1206
Connections:
- net labels removed: STRIP_GND
- wire segments 25 -> 22
Changed lines of the file:
@@
-EESchema Schematic File Version 2  date Wed 31 Oct 2012 08:56:02 PM CDT
+EESchema Schematic File Version 2
 LIBS:power
 LIBS:device
@@
 LIBS:Joe_Discrete
 LIBS:double_in_cab_breakout-cache
-EELAYER 27 0
+EELAYER 24 0
 EELAYER END
 $Descr A4 11693 8268
@@
 $EndDescr
 $Comp
-L GND #PWR03
+L GND #PWR01
 U 1 1 5068AACC
 P 2900 3650
-F 0 "#PWR03" H 2900 3650 30  0001 C CNN
+F 0 "#PWR01" H 2900 3650 30  0001 C CNN
 F 1 "GND" H 2900 3580 30  0001 C CNN
+F 2 "" H 2900 3650 60  0001 C CNN
+F 3 "" H 2900 3650 60  0001 C CNN
 	1    2900 3650
 	1    0    0    -1
 $EndComp
 $Comp
-L GND #PWR04
+L GND #PWR02
 U 1 1 5068AAD2
 P 2300 3650
-F 0 "#PWR04" H 2300 3650 30  0001 C CNN
+F 0 "#PWR02" H 2300 3650 30  0001 C CNN
 F 1 "GND" H 2300 3580 30  0001 C CNN
+F 2 "" H 2300 3650 60  0001 C CNN
+F 3 "" H 2300 3650 60  0001 C CNN
 	1    2300 3650
 	1    0    0    -1
 $EndComp
 $Comp
-L +24V #PWR05
+L +24V #PWR03
 U 1 1 5068AAE2
 P 2300 3250
-F 0 "#PWR05" H 2300 3200 20  0001 C CNN
+F 0 "#PWR03" H 2300 3200 20  0001 C CNN
 F 1 "+24V" H 2300 3350 30  0000 C CNN
+F 2 "" H 2300 3250 60  0001 C CNN
+F 3 "" H 2300 3250 60  0001 C CNN
 	1    2300 3250
 	1    0    0    -1
 $EndComp
 $Comp
-L +24V #PWR06
+L +24V #PWR04
 U 1 1 5068AAE8
 P 2900 3250
-F 0 "#PWR06" H 2900 3200 20  0001 C CNN
+F 0 "#PWR04" H 2900 3200 20  0001 C CNN
 F 1 "+24V" H 2900 3350 30  0000 C CNN
+F 2 "" H 2900 3250 60  0001 C CNN
+F 3 "" H 2900 3250 60  0001 C CNN
 	1    2900 3250
 	1    0    0    -1
@@
 F 0 "C101" H 2350 3550 50  0000 L CNN
 F 1 "CAP_2P2UF_10P_50V_X5R_1206" H 2400 3250 50  0001 L CNN
+F 2 "" H 2300 3450 60  0001 C CNN
+F 3 "" H 2300 3450 60  0001 C CNN
 F 4 "587-2402-1-ND" H 2800 3150 60  0001 C CNN "PN"
 F 5 "2.2uF" H 2175 3500 39  0000 R BNN "Val"
@@
 F 0 "C102" H 2950 3550 50  0000 L CNN
 F 1 "CAP_2P2UF_10P_50V_X5R_1206" H 3000 3250 50  0001 L CNN
+F 2 "" H 2900 3450 60  0001 C CNN
+F 3 "" H 2900 3450 60  0001 C CNN
 F 4 "587-2402-1-ND" H 3400 3150 60  0001 C CNN "PN"
 F 5 "2.2uF" H 2775 3500 39  0000 R BNN "Val"
@@
 F 0 "P10" V 8750 3200 40  0000 C CNN
 F 1 "CONN_JST_PH_2" H 8600 3000 40  0000 C CNN
+F 2 "" H 8750 3200 60  0001 C CNN
+F 3 "" H 8750 3200 60  0001 C CNN
 F 4 "455-1749-1-ND" H 8750 2900 60  0001 C CNN "PN"
 	1    8750 3200
@@
 F 0 "P11" V 7750 3200 40  0000 C CNN
 F 1 "CONN_JST_PH_2" H 7600 3000 40  0000 C CNN
+F 2 "" H 7750 3200 60  0001 C CNN
+F 3 "" H 7750 3200 60  0001 C CNN
 F 4 "455-1749-1-ND" H 7750 2900 60  0001 C CNN "PN"
 	1    7750 3200
@@
 F 0 "P13" V 8750 3800 40  0000 C CNN
 F 1 "CONN_JST_PH_2" H 8600 3600 40  0000 C CNN
+F 2 "" H 8750 3800 60  0001 C CNN
+F 3 "" H 8750 3800 60  0001 C CNN
 F 4 "455-1749-1-ND" H 8750 3500 60  0001 C CNN "PN"
 	1    8750 3800
@@
 F 0 "P14" V 7750 3800 40  0000 C CNN
 F 1 "CONN_JST_PH_2" H 7600 3600 40  0000 C CNN
+F 2 "" H 7750 3800 60  0001 C CNN
+F 3 "" H 7750 3800 60  0001 C CNN
 F 4 "455-1749-1-ND" H 7750 3500 60  0001 C CNN "PN"
 	1    7750 3800
@@
 F 0 "P16" V 6650 5100 40  0000 C CNN
 F 1 "CONN_JST_PH_2" H 6500 4900 40  0000 C CNN
+F 2 "" H 6650 5100 60  0001 C CNN
+F 3 "" H 6650 5100 60  0001 C CNN
 F 4 "455-1749-1-ND" H 6650 4800 60  0001 C CNN "PN"
 	1    6650 5100
@@
 F 0 "P17" V 7650 5100 40  0000 C CNN
 F 1 "CONN_JST_PH_2" H 7500 4900 40  0000 C CNN
+F 2 "" H 7650 5100 60  0001 C CNN
+F 3 "" H 7650 5100 60  0001 C CNN
 F 4 "455-1749-1-ND" H 7650 4800 60  0001 C CNN "PN"
 	1    7650 5100
@@
 $EndComp
 $Comp
-L GND #PWR09
+L GND #PWR05
 U 1 1 508349E0
 P 5850 2050
-F 0 "#PWR09" H 5850 2050 30  0001 C CNN
+F 0 "#PWR05" H 5850 2050 30  0001 C CNN
 F 1 "GND" H 5850 1980 30  0001 C CNN
+F 2 "" H 5850 2050 60  0001 C CNN
+F 3 "" H 5850 2050 60  0001 C CNN
 	1    5850 2050
 	-1   0    0    1
 $EndComp
 $Comp
-L GND #PWR010
+L GND #PWR06
 U 1 1 508349F0
 P 6050 2050
-F 0 "#PWR010" H 6050 2050 30  0001 C CNN
+F 0 "#PWR06" H 6050 2050 30  0001 C CNN
 F 1 "GND" H 6050 1980 30  0001 C CNN
+F 2 "" H 6050 2050 60  0001 C CNN
+F 3 "" H 6050 2050 60  0001 C CNN
 	1    6050 2050
 	-1   0    0    1
 $EndComp
 $Comp
-L +24V #PWR011
+L +24V #PWR07
 U 1 1 508349F6
 P 5650 2050
-F 0 "#PWR011" H 5650 2000 20  0001 C CNN
+F 0 "#PWR07" H 5650 2000 20  0001 C CNN
 F 1 "+24V" H 5650 2150 30  0000 C CNN
+F 2 "" H 5650 2050 60  0001 C CNN
+F 3 "" H 5650 2050 60  0001 C CNN
 	1    5650 2050
 	1    0    0    -1
 $EndComp
 $Comp
-L +24V #PWR012
+L +24V #PWR08
 U 1 1 508349FC
 P 6250 2050
-F 0 "#PWR012" H 6250 2000 20  0001 C CNN
+F 0 "#PWR08" H 6250 2000 20  0001 C CNN
 F 1 "+24V" H 6250 2150 30  0000 C CNN
+F 2 "" H 6250 2050 60  0001 C CNN
+F 3 "" H 6250 2050 60  0001 C CNN
 	1    6250 2050
 	1    0    0    -1
 $EndComp
 $Comp
-L +24V #PWR013
+L +24V #PWR09
 U 1 1 5088A59B
 P 7200 2900
-F 0 "#PWR013" H 7200 2850 20  0001 C CNN
+F 0 "#PWR09" H 7200 2850 20  0001 C CNN
 F 1 "+24V" H 7200 3000 30  0000 C CNN
+F 2 "" H 7200 2900 60  0001 C CNN
+F 3 "" H 7200 2900 60  0001 C CNN
 	1    7200 2900
 	1    0    0    -1
@@
 	7200 5000 7000 5000
 $Comp
-L GND #PWR014
+L GND #PWR010
 U 1 1 5088A629
 P 7200 5400
-F 0 "#PWR014" H 7200 5400 30  0001 C CNN
+F 0 "#PWR010" H 7200 5400 30  0001 C CNN
 F 1 "GND" H 7200 5330 30  0001 C CNN
+F 2 "" H 7200 5400 60  0001 C CNN
+F 3 "" H 7200 5400 60  0001 C CNN
 	1    7200 5400
 	1    0    0    -1
@@
 	7200 5200 7200 5400
 $Comp
-L GND #PWR015
+L GND #PWR011
 U 1 1 5088A6E6
 P 8200 5400
-F 0 "#PWR015" H 8200 5400 30  0001 C CNN
+F 0 "#PWR011" H 8200 5400 30  0001 C CNN
 F 1 "GND" H 8200 5330 30  0001 C CNN
+F 2 "" H 8200 5400 60  0001 C CNN
+F 3 "" H 8200 5400 60  0001 C CNN
 	1    8200 5400
 	1    0    0    -1
 $EndComp
 $Comp
-L +24V #PWR016
+L +24V #PWR012
 U 1 1 5088A6EC
 P 8200 2900
-F 0 "#PWR016" H 8200 2850 20  0001 C CNN
+F 0 "#PWR012" H 8200 2850 20  0001 C CNN
 F 1 "+24V" H 8200 3000 30  0000 C CNN
+F 2 "" H 8200 2900 60  0001 C CNN
+F 3 "" H 8200 2900 60  0001 C CNN
 	1    8200 2900
 	1    0    0    -1
@@
 Text Label 8200 3700 1    40   ~ 0
 STRIP2_12V
-Wire Wire Line
-	8200 5000 8200 4800
-Wire Wire Line
-	8200 4800 7200 4800
-Wire Wire Line
-	7200 4800 7200 5000
-Wire Wire Line
-	7700 4100 7700 4800
-Connection ~ 7700 4800
-Wire Wire Line
-	8200 3900 8200 4100
-Wire Wire Line
-	8200 4100 7200 4100
-Wire Wire Line
-	7200 4100 7200 3900
-Connection ~ 7700 4100
-Text Label 7700 4650 1    40   ~ 0
-STRIP_GND
 $Comp
 L CONN_TERM_BLOCK_2POS_3P5MM P100
@@
 F 0 "P100" V 5750 2400 40  0000 C CNN
 F 1 "CONN_TERM_BLOCK_2POS_3P5MM" H 5700 2650 40  0001 C CNN
+F 2 "" H 5750 2400 60  0001 C CNN
+F 3 "" H 5750 2400 60  0001 C CNN
 F 4 "A98036-ND" H 5750 2100 60  0001 C CNN "PN"
 F 5 "TRM_BLK_2" H 5450 2200 40  0000 L BNN "Name"
@@
 F 0 "P101" V 6150 2400 40  0000 C CNN
 F 1 "CONN_TERM_BLOCK_2POS_3P5MM" H 6100 2650 40  0001 C CNN
+F 2 "" H 6150 2400 60  0001 C CNN
+F 3 "" H 6150 2400 60  0001 C CNN
 F 4 "A98036-ND" H 6150 2100 60  0001 C CNN "PN"
 F 5 "TRM_BLK_2" H 5850 2200 40  0000 L BNN "Name"
@@
 	0    1    1    0
 $EndComp
+$Comp
+L RES_0_0P_1V4_1206 R1001
+U 1 1 521BC944
+P 7700 4550
+F 0 "R1001" V 7805 4550 50  0000 C CNN
+F 1 "RES_0_0P_1V4_1206" H 7175 4700 50  0001 C CNN
+F 2 "" H 7700 4550 60  0000 C CNN
+F 3 "" H 7700 4550 60  0000 C CNN
+F 4 "CR1206-J/-000ELFCT-ND" H 7080 4775 60  0001 C CNN "PN"
+F 5 "0" H 7630 4600 39  0000 R BNN "Val"
+F 6 "1206" H 7630 4450 39  0000 R BNN "Package"
+F 7 "0%" H 7630 4550 39  0000 R BNN "Tol"
+F 8 "1/4" H 7630 4500 39  0000 R BNN "Power"
+	1    7700 4550
+	0    -1   -1   0
+$EndComp
+Wire Wire Line
+	8200 3900 8200 5000
+Wire Wire Line
+	7200 3900 7200 5000
+Wire Wire Line
+	7450 4550 7200 4550
+Connection ~ 7200 4550
+Wire Wire Line
+	7950 4550 8200 4550
+Connection ~ 8200 4550
 $EndSCHEMATC
