File: boards/main_adjustment_board/main_adjustment_board.sch (KiCad schematic (older format))
At the start: 21 parts, among them P101 CONN_5X2, P102 CONN_1, P103 CONN_1, P104 CONN_1, P105 CONN_1, SW101 SW_PB_MJTP1230, SW102 SW_PB_MJTP1230, SW103 SW_PB_MJTP1230

Commit message: Modifications
Connections:
- wire segments 33 -> 29
Changed lines of the file:
@@
-EESchema Schematic File Version 2  date Sun 24 Mar 2013 05:40:36 PM CDT
+EESchema Schematic File Version 2
 LIBS:power
 LIBS:device
@@
 LIBS:Joe_Discrete
 LIBS:main_adjustment_board-cache
-EELAYER 27 0
+EELAYER 24 0
 EELAYER END
 $Descr A4 11693 8268
@@
 L POT_10K_SLIDER RV101
 U 1 1 514F1C4E
-P 5050 3850
-F 0 "RV101" V 5050 3850 50  0000 C CNN
-F 1 "POT_10K_SLIDER" V 5250 3850 50  0001 C CNN
-F 2 "" H 5050 3850 60  0001 C CNN
-F 3 "" H 5050 3850 60  0001 C CNN
-F 4 "PTA4553-2015CPB103" H 5050 4150 39  0001 C CNN "PN"
-F 5 "10K" H 5000 3900 39  0000 R BNN "Val"
-F 6 "PTA43" H 5000 3750 39  0000 R BNN "Package"
-F 7 "20%" H 5000 3850 39  0000 R BNN "Tol"
-F 8 "1/4W" H 5000 3800 39  0000 R BNN "Power"
-	1    5050 3850
+P 4500 3750
+F 0 "RV101" V 4500 3750 50  0000 C CNN
+F 1 "POT_10K_SLIDER" V 4700 3750 50  0001 C CNN
+F 2 "" H 4500 3750 60  0001 C CNN
+F 3 "" H 4500 3750 60  0001 C CNN
+F 4 "PTA4553-2015CPB103" H 4500 4050 39  0001 C CNN "PN"
+F 5 "10K" H 4450 3800 39  0000 R BNN "Val"
+F 6 "PTA43" H 4450 3650 39  0000 R BNN "Package"
+F 7 "20%" H 4450 3750 39  0000 R BNN "Tol"
+F 8 "1/4W" H 4450 3700 39  0000 R BNN "Power"
+	1    4500 3750
 	1    0    0    -1
 $EndComp
@@
 L POT_10K_SLIDER RV102
 U 1 1 514F1C82
-P 5650 3850
-F 0 "RV102" V 5650 3850 50  0000 C CNN
-F 1 "POT_10K_SLIDER" V 5850 3850 50  0001 C CNN
-F 2 "" H 5650 3850 60  0001 C CNN
-F 3 "" H 5650 3850 60  0001 C CNN
-F 4 "PTA4553-2015CPB103" H 5650 4150 39  0001 C CNN "PN"
-F 5 "10K" H 5600 3900 39  0000 R BNN "Val"
-F 6 "PTA43" H 5600 3750 39  0000 R BNN "Package"
-F 7 "20%" H 5600 3850 39  0000 R BNN "Tol"
-F 8 "1/4W" H 5600 3800 39  0000 R BNN "Power"
-	1    5650 3850
+P 5300 3750
+F 0 "RV102" V 5300 3750 50  0000 C CNN
+F 1 "POT_10K_SLIDER" V 5500 3750 50  0001 C CNN
+F 2 "" H 5300 3750 60  0001 C CNN
+F 3 "" H 5300 3750 60  0001 C CNN
+F 4 "PTA4553-2015CPB103" H 5300 4050 39  0001 C CNN "PN"
+F 5 "10K" H 5250 3800 39  0000 R BNN "Val"
+F 6 "PTA43" H 5250 3650 39  0000 R BNN "Package"
+F 7 "20%" H 5250 3750 39  0000 R BNN "Tol"
+F 8 "1/4W" H 5250 3700 39  0000 R BNN "Power"
+	1    5300 3750
 	1    0    0    -1
 $EndComp
@@
 L POT_10K_SLIDER RV103
 U 1 1 514F1C8D
-P 6250 3850
-F 0 "RV103" V 6250 3850 50  0000 C CNN
-F 1 "POT_10K_SLIDER" V 6450 3850 50  0001 C CNN
-F 2 "" H 6250 3850 60  0001 C CNN
-F 3 "" H 6250 3850 60  0001 C CNN
-F 4 "PTA4553-2015CPB103" H 6250 4150 39  0001 C CNN "PN"
-F 5 "10K" H 6200 3900 39  0000 R BNN "Val"
-F 6 "PTA43" H 6200 3750 39  0000 R BNN "Package"
-F 7 "20%" H 6200 3850 39  0000 R BNN "Tol"
-F 8 "1/4W" H 6200 3800 39  0000 R BNN "Power"
-	1    6250 3850
+P 6100 3750
+F 0 "RV103" V 6100 3750 50  0000 C CNN
+F 1 "POT_10K_SLIDER" V 6300 3750 50  0001 C CNN
+F 2 "" H 6100 3750 60  0001 C CNN
+F 3 "" H 6100 3750 60  0001 C CNN
+F 4 "PTA4553-2015CPB103" H 6100 4050 39  0001 C CNN "PN"
+F 5 "10K" H 6050 3800 39  0000 R BNN "Val"
+F 6 "PTA43" H 6050 3650 39  0000 R BNN "Package"
+F 7 "20%" H 6050 3750 39  0000 R BNN "Tol"
+F 8 "1/4W" H 6050 3700 39  0000 R BNN "Power"
+	1    6100 3750
 	1    0    0    -1
 $EndComp
@@
 L POT_10K_SLIDER RV104
 U 1 1 514F1C98
-P 6800 3850
-F 0 "RV104" V 6800 3850 50  0000 C CNN
-F 1 "POT_10K_SLIDER" V 7000 3850 50  0001 C CNN
-F 2 "" H 6800 3850 60  0001 C CNN
-F 3 "" H 6800 3850 60  0001 C CNN
-F 4 "PTA4553-2015CPB103" H 6800 4150 39  0001 C CNN "PN"
-F 5 "10K" H 6750 3900 39  0000 R BNN "Val"
-F 6 "PTA43" H 6750 3750 39  0000 R BNN "Package"
-F 7 "20%" H 6750 3850 39  0000 R BNN "Tol"
-F 8 "1/4W" H 6750 3800 39  0000 R BNN "Power"
-	1    6800 3850
+P 6900 3750
+F 0 "RV104" V 6900 3750 50  0000 C CNN
+F 1 "POT_10K_SLIDER" V 7100 3750 50  0001 C CNN
+F 2 "" H 6900 3750 60  0001 C CNN
+F 3 "" H 6900 3750 60  0001 C CNN
+F 4 "PTA4553-2015CPB103" H 6900 4050 39  0001 C CNN "PN"
+F 5 "10K" H 6850 3800 39  0000 R BNN "Val"
+F 6 "PTA43" H 6850 3650 39  0000 R BNN "Package"
+F 7 "20%" H 6850 3750 39  0000 R BNN "Tol"
+F 8 "1/4W" H 6850 3700 39  0000 R BNN "Power"
+	1    6900 3750
 	1    0    0    -1
 $EndComp
@@
 L GND #PWR01
 U 1 1 514F1CA0
-P 5050 4100
-F 0 "#PWR01" H 5050 4100 30  0001 C CNN
-F 1 "GND" H 5050 4030 30  0001 C CNN
-F 2 "" H 5050 4100 60  0001 C CNN
-F 3 "" H 5050 4100 60  0001 C CNN
-	1    5050 4100
+P 4500 4000
+F 0 "#PWR01" H 4500 4000 30  0001 C CNN
+F 1 "GND" H 4500 3930 30  0001 C CNN
+F 2 "" H 4500 4000 60  0001 C CNN
+F 3 "" H 4500 4000 60  0001 C CNN
+	1    4500 4000
 	1    0    0    -1
 $EndComp
@@
 L GND #PWR02
 U 1 1 514F1CAD
-P 5650 4100
-F 0 "#PWR02" H 5650 4100 30  0001 C CNN
-F 1 "GND" H 5650 4030 30  0001 C CNN
-F 2 "" H 5650 4100 60  0001 C CNN
-F 3 "" H 5650 4100 60  0001 C CNN
-	1    5650 4100
+P 5300 4000
+F 0 "#PWR02" H 5300 4000 30  0001 C CNN
+F 1 "GND" H 5300 3930 30  0001 C CNN
+F 2 "" H 5300 4000 60  0001 C CNN
+F 3 "" H 5300 4000 60  0001 C CNN
+	1    5300 4000
 	1    0    0    -1
 $EndComp
@@
 L GND #PWR03
 U 1 1 514F1CB3
-P 6250 4100
-F 0 "#PWR03" H 6250 4100 30  0001 C CNN
-F 1 "GND" H 6250 4030 30  0001 C CNN
-F 2 "" H 6250 4100 60  0001 C CNN
-F 3 "" H 6250 4100 60  0001 C CNN
-	1    6250 4100
+P 6100 4000
+F 0 "#PWR03" H 6100 4000 30  0001 C CNN
+F 1 "GND" H 6100 3930 30  0001 C CNN
+F 2 "" H 6100 4000 60  0001 C CNN
+F 3 "" H 6100 4000 60  0001 C CNN
+	1    6100 4000
 	1    0    0    -1
 $EndComp
@@
 L GND #PWR04
 U 1 1 514F1CB9
-P 6800 4100
-F 0 "#PWR04" H 6800 4100 30  0001 C CNN
-F 1 "GND" H 6800 4030 30  0001 C CNN
-F 2 "" H 6800 4100 60  0001 C CNN
-F 3 "" H 6800 4100 60  0001 C CNN
-	1    6800 4100
+P 6900 4000
+F 0 "#PWR04" H 6900 4000 30  0001 C CNN
+F 1 "GND" H 6900 3930 30  0001 C CNN
+F 2 "" H 6900 4000 60  0001 C CNN
+F 3 "" H 6900 4000 60  0001 C CNN
+	1    6900 4000
 	1    0    0    -1
 $EndComp
@@
 L +3.3V #PWR05
 U 1 1 514F1CDF
-P 5050 3600
-F 0 "#PWR05" H 5050 3560 30  0001 C CNN
-F 1 "+3.3V" H 5050 3710 30  0000 C CNN
-F 2 "" H 5050 3600 60  0001 C CNN
-F 3 "" H 5050 3600 60  0001 C CNN
-	1    5050 3600
+P 4500 3500
+F 0 "#PWR05" H 4500 3460 30  0001 C CNN
+F 1 "+3.3V" H 4500 3610 30  0000 C CNN
+F 2 "" H 4500 3500 60  0001 C CNN
+F 3 "" H 4500 3500 60  0001 C CNN
+	1    4500 3500
 	1    0    0    -1
 $EndComp
@@
 L +3.3V #PWR06
 U 1 1 514F1CEC
-P 5650 3600
-F 0 "#PWR06" H 5650 3560 30  0001 C CNN
-F 1 "+3.3V" H 5650 3710 30  0000 C CNN
-F 2 "" H 5650 3600 60  0001 C CNN
-F 3 "" H 5650 3600 60  0001 C CNN
-	1    5650 3600
+P 5300 3500
+F 0 "#PWR06" H 5300 3460 30  0001 C CNN
+F 1 "+3.3V" H 5300 3610 30  0000 C CNN
+F 2 "" H 5300 3500 60  0001 C CNN
+F 3 "" H 5300 3500 60  0001 C CNN
+	1    5300 3500
 	1    0    0    -1
 $EndComp
@@
 L +3.3V #PWR07
 U 1 1 514F1CF2
-P 6250 3600
-F 0 "#PWR07" H 6250 3560 30  0001 C CNN
-F 1 "+3.3V" H 6250 3710 30  0000 C CNN
-F 2 "" H 6250 3600 60  0001 C CNN
-F 3 "" H 6250 3600 60  0001 C CNN
-	1    6250 3600
+P 6100 3500
+F 0 "#PWR07" H 6100 3460 30  0001 C CNN
+F 1 "+3.3V" H 6100 3610 30  0000 C CNN
+F 2 "" H 6100 3500 60  0001 C CNN
+F 3 "" H 6100 3500 60  0001 C CNN
+	1    6100 3500
 	1    0    0    -1
 $EndComp
@@
 L +3.3V #PWR08
 U 1 1 514F1CF8
-P 6800 3600
-F 0 "#PWR08" H 6800 3560 30  0001 C CNN
-F 1 "+3.3V" H 6800 3710 30  0000 C CNN
-F 2 "" H 6800 3600 60  0001 C CNN
-F 3 "" H 6800 3600 60  0001 C CNN
-	1    6800 3600
+P 6900 3500
+F 0 "#PWR08" H 6900 3460 30  0001 C CNN
+F 1 "+3.3V" H 6900 3610 30  0000 C CNN
+F 2 "" H 6900 3500 60  0001 C CNN
+F 3 "" H 6900 3500 60  0001 C CNN
+	1    6900 3500
 	1    0    0    -1
 $EndComp
@@
 	5100 4500 5100 4900
 Wire Wire Line
-	6400 3850 6450 3850
-Wire Wire Line
-	6450 3850 6450 3300
-Wire Wire Line
-	6450 3300 7400 3300
-Wire Wire Line
-	6950 3850 7000 3850
-Wire Wire Line
-	7000 3850 7000 3400
-Wire Wire Line
-	7000 3400 7400 3400
-Wire Wire Line
-	7400 3200 5850 3200
-Wire Wire Line
-	5850 3200 5850 3850
-Wire Wire Line
-	5850 3850 5800 3850
-Wire Wire Line
-	5200 3850 5250 3850
-Wire Wire Line
-	5250 3850 5250 3100
-Wire Wire Line
-	5250 3100 7400 3100
-Text Label 7400 3100 2    60   ~ 0
+	6300 3750 6300 3200
+Wire Wire Line
+	6300 3200 7250 3200
+Wire Wire Line
+	7100 3750 7100 3300
+Wire Wire Line
+	7100 3300 7500 3300
+Wire Wire Line
+	7050 3100 5500 3100
+Wire Wire Line
+	5500 3100 5500 3750
+Wire Wire Line
+	4700 3750 4700 3000
+Wire Wire Line
+	4700 3000 6850 3000
+Text Label 6850 3000 2    60   ~ 0
 AD3
-Text Label 7400 3200 2    60   ~ 0
+Text Label 7050 3100 2    60   ~ 0
 AD4
-Text Label 7400 3300 2    60   ~ 0
+Text Label 7250 3200 2    60   ~ 0
 AD1
-Text Label 7400 3400 2    60   ~ 0
+Text Label 7500 3300 2    60   ~ 0
 AD2
 Text Label 6700 4500 2    60   ~ 0
@@
 Text Label 2600 1800 0    60   ~ 0
 SW4
+Connection ~ 4700 3750
+Connection ~ 5500 3750
+Connection ~ 6300 3750
+Connection ~ 7100 3750
 $EndSCHEMATC
