File: boards/main_control_board/main_control_board.kicad_pcb (KiCad board)
At the start: 2 copper layers, 98.8 x 101.6 mm, 123 parts, among them J101 CONN_USB_MINI_B, J102 CONN_USB_MINI_B, P1 CONN_JST_PH_4, P101 CONN_JST_PH_3, P102 CONN_JST_PH_2, P103 CONN_2, P104 CONN_5X2, P105 CONN_TERM_BLOCK_2POS_3P5MM, P106 CONN_TERM_BLOCK_2POS_3P5MM, P107 CONN_TERM_BLOCK_4POS_3P5MM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

Commit message: Modifications
Parts:
- moved C125 359.8 mm to (226.3, 126.4)
- moved D2 359.8 mm to (220.2, 106.2)
- moved P1 359.8 mm to (196.1, 155.7)
- moved R108 359.8 mm to (220.2, 116.6)
- moved R109 359.8 mm to (220.2, 114.6)
- moved C1001 359.8 mm to (208.0, 119.9)
- moved C1002 359.8 mm to (268.5, 157.0)
- moved C1008 359.8 mm to (268.5, 143.8)
- moved C104 359.8 mm to (204.1, 106.3)
- moved C107 359.8 mm to (214.1, 106.8)
- moved C110 359.8 mm to (232.2, 139.2)
- moved C112 359.8 mm to (239.5, 105.7)
- moved C12345 359.8 mm to (206.2, 113.0)
- moved D102 359.8 mm to (205.0, 96.5)
- moved D4 359.8 mm to (213.9, 150.1)
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Routing:
- net /SW2: track 16.4 -> 35.9 mm
- net /AD3: track 17.0 -> 25.9 mm
- net +24V: track 73.5 -> 78.9 mm
- net /WW_OUT: track 15.9 -> 19.9 mm, vias 2 -> 3
- net (no net): track 2.03 -> 0.00 mm, vias 1 -> 0

Commit message: main_control_board
Fixed the adjustment board ribbon cable connector pinout
Parts:
- moved C1234 7.66 mm to (229.4, 153.4)
Connections:
- P104 pad 1: /SW4 -> GND
- P104 pad 2: GND -> /SW4
- P104 pad 3: /SW1 -> +3.3V
- P104 pad 4: +3.3V -> /SW1
Routing:
- net +3.3V: track 245.0 -> 253.9 mm
- net /SW1: track 17.1 -> 20.7 mm, vias 0 -> 1
- net GND: track 170.3 -> 172.6 mm
- net /SW4: track 18.1 -> 20.3 mm
