File: boards/main_control_board/main_control_board.sch (KiCad schematic (older format))
At the start: 123 parts, among them J101 CONN_USB_MINI_B, J102 CONN_USB_MINI_B, P1 CONN_JST_PH_4, P101 CONN_JST_PH_3, P102 CONN_JST_PH_2, P103 CONN_2, P104 CONN_5X2, P105 CONN_TERM_BLOCK_2POS_3P5MM, P106 CONN_TERM_BLOCK_2POS_3P5MM, P107 CONN_TERM_BLOCK_4POS_3P5MM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

Commit message: Modifications
Changed lines of the file:
@@
-EESchema Schematic File Version 2  date Tue 26 Mar 2013 10:28:15 PM CDT
+EESchema Schematic File Version 2
 LIBS:power
 LIBS:device
@@
 LIBS:Joe_Chips
 LIBS:Joe_Discrete
-LIBS:main_Board-cache
-EELAYER 27 0
+LIBS:main_control_board-cache
+EELAYER 24 0
 EELAYER END
 $Descr C 22000 17000
@@
 Wire Wire Line
 	15900 14850 15900 14950
-Entry Wire Line
-	5150 10950 5250 11050
 $Comp
 L GND #PWR058
@@
 Wire Wire Line
 	11100 2800 10900 2800
+Entry Wire Line
+	2950 3950 3050 4050
 $EndSCHEMATC

Commit message: main_control_board
Fixed the adjustment board ribbon cable connector pinout
Changed lines of the file:
@@
-EESchema Schematic File Version 2
+EESchema Schematic File Version 2  date Wed 28 Aug 2013 08:30:11 PM CDT
 LIBS:power
 LIBS:device
@@
 LIBS:Joe_Discrete
 LIBS:main_control_board-cache
-EELAYER 24 0
+EELAYER 27 0
 EELAYER END
 $Descr C 22000 17000
@@
 Sheet 1 1
 Title ""
-Date "27 mar 2013"
+Date "29 aug 2013"
 Rev ""
 Comp ""
@@
 $EndComp
 Text Label 9200 3200 0    60   ~ 0
-AD2
+AD1
 Text Label 8500 3100 0    60   ~ 0
-AD4
+AD3
 Text Label 9100 3000 0    60   ~ 0
-SW3
+SW2
 $Comp
 L +3.3V #PWR049
@@
 F 5 "CONN_5X2" H 10500 3000 60  0001 C CNN "Name"
 	1    10500 3000
-	1    0    0    -1
+	-1   0    0    -1
 $EndComp
 Wire Wire Line
@@
 	10900 3200 11600 3200
 Text Label 11600 3000 2    60   ~ 0
-SW2
+SW3
 Text Label 11600 3100 2    60   ~ 0
-AD3
+AD4
 Text Label 11600 3200 2    60   ~ 0
-AD1
+AD2
 $Comp
 L GND #PWR0103
